Commit message: revise the crawl locomotion

File: legged_gym/resources/robots/go2/urdf/go2.urdf (robot description, URDF)
Before this commit: robot go2_description, 42 links, 41 joints
Links:
- link FL_calf: geometry collision cylinder length=0.12 radius=0.012; visual mesh filename=../meshes/calf.dae
- link FL_foot: geometry collision sphere radius=0.022; visual mesh filename=../meshes/foot.dae
- link FL_hip: geometry collision cylinder length=0.04 radius=0.046; visual mesh filename=../meshes/hip.dae
- link FL_thigh: geometry collision box size=0.213 0.0245 0.034; visual mesh filename=../meshes/thigh.dae
- link FR_calf: geometry collision cylinder length=0.12 radius=0.013; visual mesh filename=../meshes/calf_mirror.dae
- link FR_foot: geometry collision sphere radius=0.022; visual mesh filename=../meshes/foot.dae
- link FR_hip: geometry collision cylinder length=0.04 radius=0.046; visual mesh filename=../meshes/hip.dae
- link FR_thigh: geometry collision box size=0.213 0.0245 0.034; visual mesh filename=../meshes/thigh_mirror.dae
- link RL_calf: geometry collision cylinder length=0.12 radius=0.013; visual mesh filename=../meshes/calf.dae
- link RL_foot: geometry collision sphere radius=0.022; visual mesh filename=../meshes/foot.dae
- link RL_hip: geometry collision cylinder length=0.04 radius=0.046; visual mesh filename=../meshes/hip.dae
- link RL_thigh: geometry collision box size=0.213 0.0245 0.034; visual mesh filename=../meshes/thigh.dae
- link RR_calf: geometry collision cylinder length=0.12 radius=0.013; visual mesh filename=../meshes/calf_mirror.dae
- link RR_foot: geometry collision sphere radius=0.022; visual mesh filename=../meshes/foot.dae
- link RR_hip: geometry collision cylinder length=0.04 radius=0.046; visual mesh filename=../meshes/hip.dae
- link RR_thigh: geometry collision box size=0.213 0.0245 0.034; visual mesh filename=../meshes/thigh_mirror.dae
- link base: geometry collision box size=0.3762 0.0935 0.114; visual mesh filename=../meshes/base.dae

Commit message: change the go2 urdf files

File: legged_gym/resources/robots/go2/urdf/go2.urdf (robot description, URDF)
Before this commit: robot go2_description, 42 links, 41 joints
Links:
- removed link FL_calf_rotor
- removed link FL_hip_rotor
- removed link FL_thigh_rotor
- removed link FR_calf_rotor
- removed link FR_hip_rotor
- removed link FR_thigh_rotor
- removed link RL_calf_rotor
- removed link RL_hip_rotor
- removed link RL_thigh_rotor
- removed link RR_calf_rotor
- removed link RR_hip_rotor
- removed link RR_thigh_rotor
- removed link front_camera
- link FL_calf: geometry collision cylinder length=0.12 radius=0.012; visual mesh filename=../dae/calf.dae
- link FL_foot: geometry collision sphere radius=0.022; visual mesh filename=../dae/foot.dae
- link FL_hip: geometry collision cylinder length=0.04 radius=0.046; visual mesh filename=../dae/hip.dae
- link FL_thigh: geometry collision box size=0.11 0.0245 0.034; visual mesh filename=../dae/thigh.dae
- link FR_calf: geometry collision cylinder length=0.12 radius=0.013; visual mesh filename=../dae/calf_mirror.dae
- link FR_foot: geometry collision sphere radius=0.022; visual mesh filename=../dae/foot.dae
- link FR_hip: geometry collision cylinder length=0.04 radius=0.046; visual mesh filename=../dae/hip.dae
- link FR_thigh: geometry collision box size=0.11 0.0245 0.034; visual mesh filename=../dae/thigh_mirror.dae
- link RL_calf: geometry collision cylinder length=0.12 radius=0.013; visual mesh filename=../dae/calf.dae
- link RL_foot: geometry collision sphere radius=0.022; visual mesh filename=../dae/foot.dae
- link RL_hip: geometry collision cylinder length=0.04 radius=0.046; visual mesh filename=../dae/hip.dae
- link RL_thigh: geometry collision box size=0.11 0.0245 0.034; visual mesh filename=../dae/thigh.dae
- link RR_calf: geometry collision cylinder length=0.12 radius=0.013; visual mesh filename=../dae/calf_mirror.dae
- link RR_foot: geometry collision sphere radius=0.022; visual mesh filename=../dae/foot.dae
- link RR_hip: geometry collision cylinder length=0.04 radius=0.046; visual mesh filename=../dae/hip.dae
- link RR_thigh: geometry collision box size=0.11 0.0245 0.034; visual mesh filename=../dae/thigh_mirror.dae
- link base: geometry collision box size=0.3762 0.0935 0.114; visual mesh filename=../dae/base.dae
Joints:
- removed joint FL_calf_rotor_joint
- removed joint FL_hip_rotor_joint
- removed joint FL_thigh_rotor_joint
- removed joint FR_calf_rotor_joint
- removed joint FR_hip_rotor_joint
- removed joint FR_thigh_rotor_joint
- removed joint RL_calf_rotor_joint
- removed joint RL_hip_rotor_joint
- removed joint RL_thigh_rotor_joint
- removed joint RR_calf_rotor_joint
- removed joint RR_hip_rotor_joint
- removed joint RR_thigh_rotor_joint
- removed joint front_camera_joint
- joint FL_calf_joint: limit lower=-2.7227 upper=-0.83776 effort=45.43 velocity=15.70 -> lower=-2.7227 upper=-0.83776 effort=35.55 velocity=20.07
- joint FR_calf_joint: limit lower=-2.7227 upper=-0.83776 effort=45.43 velocity=15.70 -> lower=-2.7227 upper=-0.83776 effort=35.55 velocity=20.07
- joint RL_calf_joint: limit lower=-2.7227 upper=-0.83776 effort=45.43 velocity=15.70 -> lower=-2.7227 upper=-0.83776 effort=35.55 velocity=20.07
- joint RR_calf_joint: limit lower=-2.7227 upper=-0.83776 effort=45.43 velocity=15.70 -> lower=-2.7227 upper=-0.83776 effort=35.55 velocity=20.07
